File: Hardware/HBridge/HBridge.kicad_sch (KiCad schematic)
At the start: 30 parts, among them IC1 SP8M4HZGTB, IC2 SP8M4HZGTB, J1 Conn_01x03_Pin, J2 Conn_01x04_Pin, U1 TC4427xOA, U2 TC4427xOA

Commit message: Add Schottky diode component to HBridge schematic
- Introduced a new Schottky diode symbol with reference designators D5 and D6.
- Updated properties including Value, Footprint, and Description for the new diode.
- Added necessary junctions and wires to integrate the diode into the existing circuit.
- Ensured the new component is included in the BOM and is visible on the board.
Parts:
- added D5, D6: D_Schottky, Package_TO_SOT_THT:TO-220-2_Vertical, symbol Device:D_Schottky
Connections:
- net O1: now also D5.2 (A)
- net O2: now also D6.2 (A)
- net Vm: now also D5.1 (K), D6.1 (K)
Changed lines of the file:
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@@
 	)
 	(junction
+		(at 200.66 138.43)
+		(diameter 0)
+		(color 0 0 0 0)
+	)
+	(junction
+		(at 200.66 82.55)
+		(diameter 0)
+		(color 0 0 0 0)
+	)
+	(junction
 		(at 81.28 113.03)
 		(diameter 0)
@@
 	(wire
 		(pts
+			(xy 175.26 97.79) (xy 200.66 97.79)
+		)
+		(stroke
+			(width 0)
+			(type default)
+		)
+	)
+	(wire
+		(pts
 			(xy 52.07 115.57) (xy 63.5 115.57)
 		)
@@
 	(wire
 		(pts
+			(xy 200.66 138.43) (xy 207.01 138.43)
+		)
+		(stroke
+			(width 0)
+			(type default)
+		)
+	)
+	(wire
+		(pts
 			(xy 69.85 142.24) (xy 72.39 142.24)
 		)
@@
 	(wire
 		(pts
-			(xy 55.88 59.69) (xy 67.31 59.69)
+			(xy 200.66 82.55) (xy 210.82 82.55)
 		)
 		(stroke
@@
 	(wire
 		(pts
-			(xy 120.65 137.16) (xy 125.73 137.16)
+			(xy 55.88 59.69) (xy 67.31 59.69)
 		)
 		(stroke
@@
 	(wire
 		(pts
-			(xy 138.43 80.01) (xy 138.43 97.79)
+			(xy 120.65 137.16) (xy 125.73 137.16)
 		)
 		(stroke
@@
 	(wire
 		(pts
-			(xy 198.12 82.55) (xy 210.82 82.55)
+			(xy 198.12 82.55) (xy 200.66 82.55)
 		)
 		(stroke
@@
 	(wire
 		(pts
+			(xy 167.64 97.79) (xy 138.43 97.79)
+		)
+		(stroke
+			(width 0)
+			(type default)
+		)
+	)
+	(wire
+		(pts
 			(xy 125.73 137.16) (xy 125.73 138.43)
 		)
@@
 	(wire
 		(pts
-			(xy 198.12 138.43) (xy 207.01 138.43)
+			(xy 198.12 138.43) (xy 200.66 138.43)
 		)
 		(stroke
@@
 	(wire
 		(pts
+			(xy 172.72 153.67) (xy 200.66 153.67)
+		)
+		(stroke
+			(width 0)
+			(type default)
+		)
+	)
+	(wire
+		(pts
 			(xy 107.95 97.79) (xy 101.6 97.79)
 		)
@@
 	(wire
 		(pts
+			(xy 200.66 97.79) (xy 200.66 82.55)
+		)
+		(stroke
+			(width 0)
+			(type default)
+		)
+	)
+	(wire
+		(pts
+			(xy 200.66 153.67) (xy 200.66 138.43)
+		)
+		(stroke
+			(width 0)
+			(type default)
+		)
+	)
+	(wire
+		(pts
 			(xy 53.34 134.62) (xy 53.34 143.51)
 		)
@@
 	(wire
 		(pts
+			(xy 134.62 153.67) (xy 165.1 153.67)
+		)
+		(stroke
+			(width 0)
+			(type default)
+		)
+	)
+	(wire
+		(pts
 			(xy 63.5 113.03) (xy 63.5 115.57)
 		)
@@
 	(wire
 		(pts
+			(xy 138.43 80.01) (xy 138.43 97.79)
+		)
+		(stroke
+			(width 0)
+			(type default)
+		)
+	)
+	(wire
+		(pts
 			(xy 129.54 72.39) (xy 129.54 77.47)
 		)
@@
 	)
 	(symbol
+		(lib_id "Device:D_Schottky")
+		(at 168.91 153.67 0)
+		(unit 1)
+		(exclude_from_sim no)
+		(in_bom yes)
+		(on_board yes)
+		(dnp no)
+		(fields_autoplaced yes)
+		(property "Reference" "D6"
+			(at 168.5925 147.32 0)
+			(effects
+				(font
+					(size 1.27 1.27)
+				)
+			)
+		)
+		(property "Value" "D_Schottky"
+			(at 168.5925 149.86 0)
+			(effects
+				(font
+					(size 1.27 1.27)
+				)
+			)
+		)
+		(property "Footprint" "Package_TO_SOT_THT:TO-220-2_Vertical"
+			(at 168.91 153.67 0)
+			(effects
+				(font
+					(size 1.27 1.27)
+				)
+				(hide yes)
+			)
+		)
+		(property "Datasheet" "~"
+			(at 168.91 153.67 0)
+			(effects
+				(font
+					(size 1.27 1.27)
+				)
+				(hide yes)
+			)
+		)
+		(property "Description" "Schottky diode"
+			(at 168.91 153.67 0)
+			(effects
+				(font
+					(size 1.27 1.27)
+				)
+				(hide yes)
+			)
+		)
+		(pin "1"
+		)
+		(pin "2"
+		)
+		(instances
+			(project ""
+				(path "/cae0d301-ea33-4e3c-a36c-9b3f252ab890"
+					(reference "D6")
+					(unit 1)
+				)
+			)
+		)
+	)
+	(symbol
 		(lib_id "Device:R")
 		(at 60.96 123.19 90)
@@
 					(unit 1)
 				)
+			)
+		)
+	)
+	(symbol
+		(lib_id "Device:D_Schottky")
+		(at 171.45 97.79 0)
+		(unit 1)
+		(exclude_from_sim no)
+		(in_bom yes)
+		(on_board yes)
+		(dnp no)
+		(fields_autoplaced yes)
+		(property "Reference" "D5"
+			(at 171.1325 91.44 0)
+			(effects
+				(font
+					(size 1.27 1.27)
+				)
+			)
+		)
+		(property "Value" "D_Schottky"
+			(at 171.1325 93.98 0)
+			(effects
+				(font
+					(size 1.27 1.27)
+				)
+			)
+		)
+		(property "Footprint" "Package_TO_SOT_THT:TO-220-2_Vertical"
+			(at 171.45 97.79 0)
+			(effects
+				(font
+					(size 1.27 1.27)
+				)
+				(hide yes)
+			)
+		)
+		(property "Datasheet" "~"
+			(at 171.45 97.79 0)
+			(effects
+				(font
+					(size 1.27 1.27)
+				)
+				(hide yes)
+			)
+		)
+		(property "Description" "Schottky diode"
+			(at 171.45 97.79 0)
+			(effects
+				(font
+					(size 1.27 1.27)
+				)
+				(hide yes)
+			)
+		)
+		(pin "1"
+		)
+		(pin "2"
+		)
+		(instances
+			(project ""
+				(path "/cae0d301-ea33-4e3c-a36c-9b3f252ab890"
+					(reference "D5")
+					(unit 1)
+				)
